File: ECAD/Keyboard12/Keyboard12/Keyboard12.kicad_pcb (KiCad board)
At the start: 4 copper layers, 95.2 x 76.2 mm, 68 parts, among them J1 CHAIN_IN_PADS, J2 CHAIN_OUT_PADS, J3 CHAIN_IN_PADS, J4 CHAIN_OUT_PADS, U1 ADS7953SDBT, U10 DRV5056A3QDBZx Lekker, U11 DRV5056A3QDBZx Lekker, U12 DRV5056A3QDBZx Lekker, U13 DRV5056A3QDBZx Lekker, U14 DRV5056A3QDBZx Lekker, U2 REF5025AIDR, U3 DRV5056A3QDBZx Lekker, U4 DRV5056A3QDBZx Lekker, U5 DRV5056A3QDBZx Lekker, U6 DRV5056A3QDBZx Lekker, U7 DRV5056A3QDBZx Lekker, U8 DRV5056A3QDBZx Lekker, U9 DRV5056A3QDBZx Lekker

Commit message: added files before cleanup
Parts:
- added REF**: MountingHole_3.2mm_M3, MountingHole:MountingHole_3.2mm_M3, F.Cu at (166.7, 128.6)
- added REF**: MountingHole_3.2mm_M3, MountingHole:MountingHole_3.2mm_M3, F.Cu at (109.5, 128.6)
- added REF**: MountingHole_3.2mm_M3, MountingHole:MountingHole_3.2mm_M3, F.Cu at (109.5, 90.5)
- moved R14 12.5 mm to (94.0, 88.0)
- moved U1 2.92 mm to (119.5, 83.5)
- moved R13 2.55 mm to (113.0, 86.0)
- moved U2 1.58 mm to (100.5, 84.0)
- moved C7 0.71 mm to (107.0, 86.0)
